File: Hardware/PCB/kdlfo/kdlfo.kicad_sch (KiCad schematic)
At the start: 31 parts, among them J1 3_pin_Molex_header, J10 AudioJack2, J11 3_pin_Molex_connector, J12 3_pin_Molex_connector, J13 3_pin_Molex_connector, J14 3_pin_Molex_connector, J15 Synth_power_2x5, J2 3_pin_Molex_header, J3 3_pin_Molex_header, J4 3_pin_Molex_header, J5 AudioJack2, J6 AudioJack2, J7 AudioJack2, J8 AudioJack2, J9 AudioJack2

Commit message: BOM
Parts:
- C1: SKU (none) -> A-984; Vendor (none) -> Tayda
- C2: SKU A-4223 -> A-4532
- C3, C4: SKU (none) -> A-4349
- D1, D2: SKU (none) -> A-159; Vendor (none) -> Tayda
- J10, J5, J6, J7, J8, J9: footprint (none) -> ao_tht:Jack_6.35mm_PJ_629HAN_slots; SKU (none) -> A-1121; Vendor (none) -> Tayda
- RV1, RV2, RV3, RV4: SKU (none) -> A-1984
Changed lines of the file:
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@@
+      (effects (font (size 1.27 1.27)) hide)
+    )
+    (property "SKU" "A-159" (id 4) (at 217.17 134.62 0)
+      (effects (font (size 1.27 1.27)) hide)
+    )
+    (property "Vendor" "Tayda" (id 5) (at 217.17 134.62 0)
       (effects (font (size 1.27 1.27)) hide)
     )
@@
       (effects (font (size 1.27 1.27)) hide)
     )
+    (property "Description" "Electrolytic capacitor, pitch 2.5 mm" (id 5) (at 243.84 135.89 0)
+      (effects (font (size 1.27 1.27)) hide)
+    )
+    (property "SKU" "A-4349" (id 6) (at 243.84 135.89 0)
+      (effects (font (size 1.27 1.27)) hide)
+    )
     (pin "1")
     (pin "2")
@@
     )
     (property "Vendor" "Tayda" (id 4) (at 243.84 143.51 0)
+      (effects (font (size 1.27 1.27)) hide)
+    )
+    (property "Description" "Electrolytic capacitor, pitch 2.5 mm" (id 5) (at 243.84 143.51 0)
+      (effects (font (size 1.27 1.27)) hide)
+    )
+    (property "SKU" "A-4349" (id 6) (at 243.84 143.51 0)
       (effects (font (size 1.27 1.27)) hide)
     )
@@
       (effects (font (size 1.27 1.27)) hide)
     )
+    (property "SKU" "A-159" (id 4) (at 217.17 144.78 0)
+      (effects (font (size 1.27 1.27)) hide)
+    )
+    (property "Vendor" "Tayda" (id 5) (at 217.17 144.78 0)
+      (effects (font (size 1.27 1.27)) hide)
+    )
     (pin "1")
     (pin "2")
@@
     )
     (property "Vendor" "Tayda" (id 4) (at 161.925 29.845 0)
+      (effects (font (size 1.27 1.27)) hide)
+    )
+    (property "SKU" "A-1984" (id 5) (at 161.925 29.845 0)
       (effects (font (size 1.27 1.27)) hide)
     )
@@
       (effects (font (size 1.27 1.27)) hide)
     )
+    (property "SKU" "A-1984" (id 5) (at 161.925 47.625 0)
+      (effects (font (size 1.27 1.27)) hide)
+    )
     (pin "1")
     (pin "2")
@@
       (effects (font (size 1.27 1.27)) (justify right))
     )
-    (property "Footprint" "" (id 2) (at 121.285 57.15 0)
+    (property "Footprint" "ao_tht:Jack_6.35mm_PJ_629HAN_slots" (id 2) (at 121.285 57.15 0)
       (effects (font (size 1.27 1.27)) hide)
     )
     (property "Datasheet" "~" (id 3) (at 121.285 57.15 0)
+      (effects (font (size 1.27 1.27)) hide)
+    )
+    (property "Description" "1/4\" phone jack, vertical" (id 4) (at 121.285 57.15 0)
+      (effects (font (size 1.27 1.27)) hide)
+    )
+    (property "SKU" "A-1121" (id 5) (at 121.285 57.15 0)
+      (effects (font (size 1.27 1.27)) hide)
+    )
+    (property "Vendor" "Tayda" (id 6) (at 121.285 57.15 0)
       (effects (font (size 1.27 1.27)) hide)
     )
@@
       (effects (font (size 1.27 1.27)) hide)
     )
+    (property "SKU" "A-1984" (id 5) (at 161.925 99.695 0)
+      (effects (font (size 1.27 1.27)) hide)
+    )
     (pin "1")
     (pin "2")
@@
       (effects (font (size 1.27 1.27)) (justify right))
     )
-    (property "Footprint" "" (id 2) (at 120.65 151.765 0)
+    (property "Footprint" "ao_tht:Jack_6.35mm_PJ_629HAN_slots" (id 2) (at 120.65 151.765 0)
       (effects (font (size 1.27 1.27)) hide)
     )
     (property "Datasheet" "~" (id 3) (at 120.65 151.765 0)
+      (effects (font (size 1.27 1.27)) hide)
+    )
+    (property "Description" "1/4\" phone jack, vertical" (id 4) (at 120.65 151.765 0)
+      (effects (font (size 1.27 1.27)) hide)
+    )
+    (property "SKU" "A-1121" (id 5) (at 120.65 151.765 0)
+      (effects (font (size 1.27 1.27)) hide)
+    )
+    (property "Vendor" "Tayda" (id 6) (at 120.65 151.765 0)
       (effects (font (size 1.27 1.27)) hide)
     )
@@
       (effects (font (size 1.27 1.27)) hide)
     )
-    (property "SKU" "A-4223" (id 5) (at 49.53 123.19 0)
+    (property "SKU" "A-4532" (id 5) (at 49.53 123.19 0)
+      (effects (font (size 1.27 1.27)) hide)
+    )
+    (property "Description" "Electrolytic capacitor, pitch 2.0 mm" (id 6) (at 49.53 123.19 0)
       (effects (font (size 1.27 1.27)) hide)
     )
@@
     )
     (property "Vendor" "Tayda" (id 4) (at 161.925 117.475 0)
+      (effects (font (size 1.27 1.27)) hide)
+    )
+    (property "SKU" "A-1984" (id 5) (at 161.925 117.475 0)
       (effects (font (size 1.27 1.27)) hide)
     )
@@
       (effects (font (size 1.27 1.27)) hide)
     )
+    (property "Description" "Polyester capacitor" (id 4) (at 49.53 53.34 0)
+      (effects (font (size 1.27 1.27)) hide)
+    )
+    (property "SKU" "A-984" (id 5) (at 49.53 53.34 0)
+      (effects (font (size 1.27 1.27)) hide)
+    )
+    (property "Vendor" "Tayda" (id 6) (at 49.53 53.34 0)
+      (effects (font (size 1.27 1.27)) hide)
+    )
     (pin "1")
     (pin "2")
@@
       (effects (font (size 1.27 1.27)) (justify right))
     )
-    (property "Footprint" "" (id 2) (at 120.65 69.85 0)
+    (property "Footprint" "ao_tht:Jack_6.35mm_PJ_629HAN_slots" (id 2) (at 120.65 69.85 0)
       (effects (font (size 1.27 1.27)) hide)
     )
     (property "Datasheet" "~" (id 3) (at 120.65 69.85 0)
+      (effects (font (size 1.27 1.27)) hide)
+    )
+    (property "Description" "1/4\" phone jack, vertical" (id 4) (at 120.65 69.85 0)
+      (effects (font (size 1.27 1.27)) hide)
+    )
+    (property "SKU" "A-1121" (id 5) (at 120.65 69.85 0)
+      (effects (font (size 1.27 1.27)) hide)
+    )
+    (property "Vendor" "Tayda" (id 6) (at 120.65 69.85 0)
       (effects (font (size 1.27 1.27)) hide)
     )
@@
       (effects (font (size 1.27 1.27)) (justify right))
     )
-    (property "Footprint" "" (id 2) (at 120.65 127 0)
+    (property "Footprint" "ao_tht:Jack_6.35mm_PJ_629HAN_slots" (id 2) (at 120.65 127 0)
       (effects (font (size 1.27 1.27)) hide)
     )
     (property "Datasheet" "~" (id 3) (at 120.65 127 0)
+      (effects (font (size 1.27 1.27)) hide)
+    )
+    (property "Description" "1/4\" phone jack, vertical" (id 4) (at 120.65 127 0)
+      (effects (font (size 1.27 1.27)) hide)
+    )
+    (property "SKU" "A-1121" (id 5) (at 120.65 127 0)
+      (effects (font (size 1.27 1.27)) hide)
+    )
+    (property "Vendor" "Tayda" (id 6) (at 120.65 127 0)
       (effects (font (size 1.27 1.27)) hide)
     )
@@
       (effects (font (size 1.27 1.27)) (justify right))
     )
-    (property "Footprint" "" (id 2) (at 120.65 81.915 0)
+    (property "Footprint" "ao_tht:Jack_6.35mm_PJ_629HAN_slots" (id 2) (at 120.65 81.915 0)
       (effects (font (size 1.27 1.27)) hide)
     )
     (property "Datasheet" "~" (id 3) (at 120.65 81.915 0)
+      (effects (font (size 1.27 1.27)) hide)
+    )
+    (property "Description" "1/4\" phone jack, vertical" (id 4) (at 120.65 81.915 0)
+      (effects (font (size 1.27 1.27)) hide)
+    )
+    (property "SKU" "A-1121" (id 5) (at 120.65 81.915 0)
+      (effects (font (size 1.27 1.27)) hide)
+    )
+    (property "Vendor" "Tayda" (id 6) (at 120.65 81.915 0)
       (effects (font (size 1.27 1.27)) hide)
     )
@@
       (effects (font (size 1.27 1.27)) (justify right))
     )
-    (property "Footprint" "" (id 2) (at 120.65 139.7 0)
+    (property "Footprint" "ao_tht:Jack_6.35mm_PJ_629HAN_slots" (id 2) (at 120.65 139.7 0)
       (effects (font (size 1.27 1.27)) hide)
     )
@@
       (effects (font (size 1.27 1.27)) hide)
     )
+    (property "Description" "1/4\" phone jack, vertical" (id 4) (at 120.65 139.7 0)
+      (effects (font (size 1.27 1.27)) hide)
+    )
+    (property "SKU" "A-1121" (id 5) (at 120.65 139.7 0)
+      (effects (font (size 1.27 1.27)) hide)
+    )
+    (property "Vendor" "Tayda" (id 6) (at 120.65 139.7 0)
+      (effects (font (size 1.27 1.27)) hide)
+    )
