File: Hardware/PCB/kdlfo/onelfo.kicad_sch (KiCad schematic)
At the start: 35 parts, among them J10 AudioJack2, J12 AudioJack2, J14 AudioJack2, Q3 2N3904, Q4 2N3904

Commit message: Reorg schematic, redo layout some more
Parts:
- removed J10, J12, J14: AudioJack2, ao_tht:Jack_6.35mm_PJ_629HAN, symbol Connector:AudioJack2
- C2: value (none) -> 220n; footprint (none) -> ao_tht:C_Rect_L7.2mm_W7.2mm_P5.00mm_FKS2_FKP2_MKS2_MKP2
- D6: value (none) -> LED_Dual_2pin; footprint (none) -> ao_tht:LED_D5.0mm
- U1: value (none) -> TL074; footprint (none) -> ao_tht:DIP-14_W7.62mm_Socket_LongPads
- U2: value (none) -> TL072
Other:
- company: (none) -> Rich Holmes / Analog Output
- title: (none) -> Variable waveshape LFO

Commit message: Fix LED
Parts:
- removed R14: 4.7k, ao_tht:R_Axial_DIN0207_L6.3mm_D2.5mm_P10.16mm_Horizontal, symbol Device:R
- added R14: RL, ao_tht:R_Axial_DIN0207_L6.3mm_D2.5mm_P10.16mm_Horizontal, symbol ao_symbols:R
- C2: value 220n -> 220n/2.2uF
Connections:
- net GND: now also R14.2; no longer U2.6 (-)
- net at C2.1, R12.2, R22.2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: now also U2.5 (+)
- net at D6.1 (KA): now also U2.6 (-), R14.1; no longer U2.5 (+)
Other:
- note added: "Choose RL for desired LED brightness, I used 1k with the BOM LED."
- moved on the sheet: C4, C5, C6, C8, D6, U1E, U2B, U2C

Commit message: Final pre fab tweaks, Gerbers
Parts:
- removed C2: 220n/2.2uF, ao_tht:C_Rect_L7.2mm_W7.2mm_P5.00mm_FKS2_FKP2_MKS2_MKP2, symbol Device:C
- D3: renamed from D2; footprint Diode_THT:D_DO-35_SOD27_P7.62mm_Horizontal -> (none)
- D4: footprint Diode_THT:D_DO-35_SOD27_P7.62mm_Horizontal -> (none)
- R2: value 100 -> (none)
- RV5: renamed from RV6; value B50K -> (none)
- RV7: renamed from RV8; value B5K -> (none)
- renumbered C4 to C5, C8 to C6, C5 to C7, C6 to C8, D6 to D5, Q3 to Q1, Q4 to Q2, R22 to R1, R4 to R10, R25 to R11, R6 to R12, R20 to R13, R10 to R14, R12 to R15, R26 to R16, R14 to R17, R29 to R3, R18 to R4, R32 to R5, R9 to R6, R19 to R7, R34 to R8, R30 to R9, RV10 to RV6
Connections:
- net GND: now also RV7.1; no longer RV7.2, RV7.3
- net SINE: now also RV7.2, RV7.3; no longer RV7.1
- net SINE_ROUND: now also RV5.3; no longer RV5.1
- net CAP1: now reaches R2.2, U1.9 (-)
- net CAP2: now reaches R1.2, R15.2, R6.2, U1.8, U2.5 (+)
- net at Q1.2 (B), R3.1: now also RV5.1; no longer RV5.3
- net at Q1.3 (C), R13.2, R4.2: now also U2.2 (-); no longer U2.3 (+)
- net at Q2.3 (C), R11.1, R7.2: now also U2.3 (+); no longer U2.2 (-)
Other:
- moved on the sheet: RV5

Commit message: Slotted jack footprints you idiot
Parts:
- D3, D4: footprint (none) -> ao_tht:D_DO-35_SOD27_P7.62mm_Horizontal
- R2: value (none) -> 100R
- RV5: value (none) -> B50k
- RV7: value (none) -> B5k
Changed lines of the file:
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@@
     (in_bom yes) (on_board yes)
     (property "Reference" "R2" (id 0) (at 91.44 43.0022 90))
-    (property "Value" "" (id 1) (at 91.44 45.3136 90))
+    (property "Value" "100R" (id 1) (at 91.44 45.3136 90))
     (property "Footprint" "ao_tht:R_Axial_DIN0207_L6.3mm_D2.5mm_P10.16mm_Horizontal" (id 2) (at 91.44 46.482 90)
       (effects (font (size 1.27 1.27)) hide)
@@
       (effects (font (size 1.27 1.27)) (justify right))
     )
-    (property "Value" "" (id 1) (at 174.7521 142.6722 0)
+    (property "Value" "B5k" (id 1) (at 174.7521 142.6722 0)
       (effects (font (size 1.27 1.27)) (justify right))
     )
@@
       (effects (font (size 1.27 1.27)) (justify right))
     )
-    (property "Value" "" (id 1) (at 83.058 127.4322 0)
+    (property "Value" "B50k" (id 1) (at 83.058 127.4322 0)
       (effects (font (size 1.27 1.27)) (justify right))
     )
@@
       (effects (font (size 1.27 1.27)) (justify right))
     )
-    (property "Footprint" "" (id 2) (at 132.715 39.37 0)
+    (property "Footprint" "ao_tht:D_DO-35_SOD27_P7.62mm_Horizontal" (id 2) (at 132.715 39.37 0)
       (effects (font (size 1.27 1.27)) hide)
     )
@@
       (effects (font (size 1.27 1.27)) (justify right))
     )
-    (property "Footprint" "" (id 2) (at 160.655 49.53 0)
-      (effects (font (size 1.27 1.27)) hide)
-    )
+    (property "Footprint" "ao_tht:D_DO-35_SOD27_P7.62mm_Horizontal" (id 2) (at 160.655 49.53 0)
+      (effects (font (size 1.27 1.27)) hide)
+    )

Commit message: BOM
Parts:
- C5, C6, C7, C8: SKU (none) -> A-553; Vendor (none) -> Tayda
- D3, D4: SKU (none) -> A-157; Vendor (none) -> Tayda
- D5: SKU (none) -> A-1050; Vendor (none) -> Tayda
- R10, R12, R15, R2, R6: Vendor (none) -> Tayda
- RV5, RV6: SKU (none) -> A-598
- RV7: SKU (none) -> A-597
- U1: SKU (none) -> A-1138; Vendor (none) -> Tayda
Changed lines of the file:
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@@
+      (effects (font (size 1.27 1.27)) hide)
+    )
+    (property "Vendor" "Tayda" (id 4) (at 91.44 48.26 0)
       (effects (font (size 1.27 1.27)) hide)
     )
@@
       (effects (font (size 1.27 1.27)) hide)
     )
+    (property "SKU" "A-597" (id 5) (at 176.53 140.97 0)
+      (effects (font (size 1.27 1.27)) hide)
+    )
     (pin "1")
     (pin "2")
@@
     )
     (property "Datasheet" "http://www.ti.com/lit/ds/symlink/tl071.pdf" (id 3) (at 133.35 71.12 0)
+      (effects (font (size 1.27 1.27)) hide)
+    )
+    (property "SKU" "A-1138" (id 4) (at 132.08 76.2 0)
+      (effects (font (size 1.27 1.27)) hide)
+    )
+    (property "Vendor" "Tayda" (id 5) (at 132.08 76.2 0)
       (effects (font (size 1.27 1.27)) hide)
     )
@@
       (effects (font (size 1.27 1.27)) hide)
     )
+    (property "SKU" "A-1050" (id 4) (at 205.74 111.76 0)
+      (effects (font (size 1.27 1.27)) hide)
+    )
+    (property "Vendor" "Tayda" (id 5) (at 205.74 111.76 0)
+      (effects (font (size 1.27 1.27)) hide)
+    )
     (pin "1")
     (pin "2")
@@
       (effects (font (size 1.27 1.27)) hide)
     )
+    (property "SKU" "A-598" (id 5) (at 81.28 125.73 0)
+      (effects (font (size 1.27 1.27)) hide)
+    )
     (pin "1")
     (pin "2")
@@
       (effects (font (size 1.27 1.27)) hide)
     )
+    (property "Description" "Ceramic capacitor, pitch 2.5 mm" (id 4) (at 229.235 42.545 0)
+      (effects (font (size 1.27 1.27)) hide)
+    )
+    (property "SKU" "A-553" (id 5) (at 229.235 42.545 0)
+      (effects (font (size 1.27 1.27)) hide)
+    )
+    (property "Vendor" "Tayda" (id 6) (at 229.235 42.545 0)
+      (effects (font (size 1.27 1.27)) hide)
+    )
     (pin "1")
     (pin "2")
@@
     )
     (property "Datasheet" "https://assets.nexperia.com/documents/data-sheet/1N4148_1N4448.pdf" (id 3) (at 128.27 39.37 0)
+      (effects (font (size 1.27 1.27)) hide)
+    )
+    (property "SKU" "A-157" (id 4) (at 128.27 39.37 0)
+      (effects (font (size 1.27 1.27)) hide)
+    )
+    (property "Vendor" "Tayda" (id 5) (at 128.27 39.37 0)
       (effects (font (size 1.27 1.27)) hide)
     )
@@
       (effects (font (size 1.27 1.27)) hide)
     )
+    (property "Vendor" "Tayda" (id 4) (at 147.32 69.85 0)
+      (effects (font (size 1.27 1.27)) hide)
+    )
     (pin "1")
     (pin "2")
@@
     )
     (property "Datasheet" "http://www.ti.com/lit/ds/symlink/tl071.pdf" (id 3) (at 97.79 78.74 0)
+      (effects (font (size 1.27 1.27)) hide)
+    )
+    (property "SKU" "A-1138" (id 4) (at 96.52 73.66 0)
+      (effects (font (size 1.27 1.27)) hide)
+    )
+    (property "Vendor" "Tayda" (id 5) (at 96.52 73.66 0)
       (effects (font (size 1.27 1.27)) hide)
     )
@@
       (effects (font (size 1.27 1.27)) hide)
     )
+    (property "Description" "Ceramic capacitor, pitch 2.5 mm" (id 4) (at 229.235 50.165 0)
+      (effects (font (size 1.27 1.27)) hide)
+    )
+    (property "SKU" "A-553" (id 5) (at 229.235 50.165 0)
+      (effects (font (size 1.27 1.27)) hide)
+    )
+    (property "Vendor" "Tayda" (id 6) (at 229.235 50.165 0)
+      (effects (font (size 1.27 1.27)) hide)
+    )
     (pin "1")
     (pin "2")
@@
       (effects (font (size 1.27 1.27)) hide)
     )
+    (property "Vendor" "Tayda" (id 4) (at 111.76 73.66 0)
+      (effects (font (size 1.27 1.27)) hide)
+    )
     (pin "1")
     (pin "2")
@@
     )
     (property "Datasheet" "http://www.ti.com/lit/ds/symlink/tl071.pdf" (id 3) (at 137.16 27.94 0)
+      (effects (font (size 1.27 1.27)) hide)
+    )
+    (property "SKU" "A-1138" (id 4) (at 138.43 33.02 0)
+      (effects (font (size 1.27 1.27)) hide)
+    )
+    (property "Vendor" "Tayda" (id 5) (at 138.43 33.02 0)
       (effects (font (size 1.27 1.27)) hide)
     )
@@
       (effects (font (size 1.27 1.27)) hide)
     )
+    (property "Description" "Ceramic capacitor, pitch 2.5 mm" (id 4) (at 228.6 73.66 0)
+      (effects (font (size 1.27 1.27)) hide)
+    )
+    (property "SKU" "A-553" (id 5) (at 228.6 73.66 0)
+      (effects (font (size 1.27 1.27)) hide)
+    )
+    (property "Vendor" "Tayda" (id 6) (at 228.6 73.66 0)
+      (effects (font (size 1.27 1.27)) hide)
+    )
     (pin "1")
     (pin "2")
@@
     )
     (property "Datasheet" "http://www.ti.com/lit/ds/symlink/tl071.pdf" (id 3) (at 165.1 38.1 0)
+      (effects (font (size 1.27 1.27)) hide)
+    )
+    (property "SKU" "A-1138" (id 4) (at 166.37 43.18 0)
+      (effects (font (size 1.27 1.27)) hide)
+    )
+    (property "Vendor" "Tayda" (id 5) (at 166.37 43.18 0)
       (effects (font (size 1.27 1.27)) hide)
     )
@@
       (effects (font (size 1.27 1.27)) hide)
     )
+    (property "Description" "Ceramic capacitor, pitch 2.5 mm" (id 4) (at 228.6 81.28 0)
+      (effects (font (size 1.27 1.27)) hide)
+    )
+    (property "SKU" "A-553" (id 5) (at 228.6 81.28 0)
+      (effects (font (size 1.27 1.27)) hide)
+    )
+    (property "Vendor" "Tayda" (id 6) (at 228.6 81.28 0)
+      (effects (font (size 1.27 1.27)) hide)
+    )
     (pin "1")
     (pin "2")
@@
       (effects (font (size 1.27 1.27)) hide)
     )
+    (property "Vendor" "Tayda" (id 4) (at 132.08 63.5 0)
+      (effects (font (size 1.27 1.27)) hide)
+    )
     (pin "1")
     (pin "2")
@@
     )
     (property "Datasheet" "https://assets.nexperia.com/documents/data-sheet/1N4148_1N4448.pdf" (id 3) (at 156.21 49.53 0)
+      (effects (font (size 1.27 1.27)) hide)
+    )
+    (property "SKU" "A-157" (id 4) (at 156.21 49.53 0)
+      (effects (font (size 1.27 1.27)) hide)
+    )
+    (property "Vendor" "Tayda" (id 5) (at 156.21 49.53 0)
       (effects (font (size 1.27 1.27)) hide)
     )
@@
     )
     (property "Datasheet" "http://www.ti.com/lit/ds/symlink/tl071.pdf" (id 3) (at 245.11 72.39 0)
+      (effects (font (size 1.27 1.27)) hide)
+    )
+    (property "SKU" "A-1138" (id 4) (at 243.84 77.47 0)
+      (effects (font (size 1.27 1.27)) hide)
+    )
+    (property "Vendor" "Tayda" (id 5) (at 243.84 77.47 0)
       (effects (font (size 1.27 1.27)) hide)
     )
@@
       (effects (font (size 1.27 1.27)) hide)
     )
+    (property "Vendor" "Tayda" (id 4) (at 158.75 90.17 0)
+      (effects (font (size 1.27 1.27)) hide)
+    )
     (pin "1")
     (pin "2")
@@
       (effects (font (size 1.27 1.27)) hide)
     )
+    (property "SKU" "A-598" (id 5) (at 110.49 151.13 0)
+      (effects (font (size 1.27 1.27)) hide)
+    )

Commit message: Fix silkscreen errors and omissions, change integ resistor, add shape resistor
Parts:
- added R35: 200R, ao_tht:R_Axial_DIN0207_L6.3mm_D2.5mm_P10.16mm_Horizontal, symbol ao_symbols:R
- C5, C6, C7, C8: SKU A-553 -> (none); Vendor Tayda -> (none)
- D3, D4: SKU A-157 -> (none); Vendor Tayda -> (none)
- D5: SKU A-1050 -> (none); Vendor Tayda -> (none)
- R10, R12, R15, R6: Vendor Tayda -> (none)
- R2: value 100R -> 300R; Vendor Tayda -> (none)
- RV5, RV6: SKU A-598 -> (none)
- RV7: SKU A-597 -> (none)
- U1: SKU A-1138 -> (none); Vendor Tayda -> (none)
Connections:
- net GND: now also R35.2
- net SHPOTCCW: now also D3.1 (K), U1.2 (-); no longer D4.2 (A), U1.6 (-)
- net SHPOTCW: now also D4.2 (A), U1.6 (-); no longer D3.1 (K), U1.2 (-)
- new net FRPOTCCW: R35.1

Commit message: Schematic annotations
Other:
- note added: "Added 200R in series with frequency pot to establish nonzero minimum frequency."
- note added: "Original had JFET based tri to sin; replaced with differential pair shaper."
- note added: "Original had inverting LED driver."
- note added: "Original value was 100R. I found this was too low for the op amps to drive and caused bad behavior; increased to 300R."
Changed lines of the file:
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@@
+    (effects (font (size 1.27 1.27)) (justify left bottom))
+  )
+  (text "Original had inverting LED driver." (at 204.47 100.33 0)
+    (effects (font (size 1.27 1.27)) (justify left bottom))
+  )
+  (text "Original value was 100R. I found this was too\nlow for the op amps to drive and caused bad\nbehavior; increased to 300R."
+    (at 45.72 43.18 0)
+    (effects (font (size 1.27 1.27)) (justify left bottom))
+  )
+  (text "Original had JFET based tri to sin; replaced \nwith differential pair shaper."
+    (at 41.91 137.16 0)
+    (effects (font (size 1.27 1.27)) (justify left bottom))
+  )
+  (text "Added 200R in series with frequency pot\nto establish nonzero minimum frequency."
+    (at 179.07 72.39 0)
     (effects (font (size 1.27 1.27)) (justify left bottom))
   )
